File: SimpleCPLD/SimpleCPLD.kicad_pcb (KiCad board)
At the start: 4 copper layers, 51.2 x 18.3 mm, 16 parts, among them P1 CONN_02X05, P2 CONN_01X17, P3 CONN_01X17, U1 EPM7064_TQFP

Commit message: Changed back silkscreen text
Other:
- board text added: "Simple CPLD rev 1.a"
- board text removed: "Stache's Simple CPLD rev 1.a"
Changed lines of the file:
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@@
   )
   (setup
-    (last_trace_width 0.381)
+    (last_trace_width 0.25)
     (user_trace_width 0.254)
     (user_trace_width 0.381)
@@
       (net 9 "Net-(TCO1-Pad1)"))
   )
-  (gr_text "Stache's Simple CPLD rev 1.a" (at 134.366 91.44) (layer B.SilkS)
+  (gr_text "Simple CPLD rev 1.a" (at 134.366 91.44) (layer B.SilkS)
     (effects (font (size 1.5 1.5) (thickness 0.3)) (justify mirror))
   )
